File: stepper_driver_PCB/usb.kicad_sch (KiCad schematic)
At the start: 4 parts, among them J5 USB-C 16P, U6 USBLC6-2SC6

Commit message: Updated PCB
Parts:
- FL1: value TDK ACM2012-900 -> TDK ACM2012-900; footprint ACM2012_900_2P_T002:ACM2012_TDK -> Marijn_KiCad:ACM2012_TDK_UPDATE
Changed lines of the file:
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@@
 			)
 		)
-		(property "Value" " TDK ACM2012-900"
+		(property "Value" "TDK ACM2012-900"
 			(at 80.01 43.942 0)
 			(effects
@@
 			)
 		)
-		(property "Footprint" "ACM2012_900_2P_T002:ACM2012_TDK"
+		(property "Footprint" "Marijn_KiCad:ACM2012_TDK_UPDATE"
 			(at 80.01 45.72 0)
 			(effects
@@
 			)
 		)
-		(property "Description" " TDK ACM2012-900-2P-T002 "
+		(property "Description" "TDK ACM2012-900-2P-T002"
 			(at 80.01 39.37 0)
 			(effects
