File: stepper_driver_PCB/stepper_driver_PCB.kicad_pcb (KiCad board)
At the start: 4 copper layers, 42.3 x 42.3 mm, 48 parts, among them J1 POWER, J2 CTRL, J3 STEPPER, J4 JTAG, J5 USB-C 16P, SW1 BTN, SW2 BTN, U1 AP7343, U3 24LC512, U4 STM32F412CEUx, U5 TMC2226-SA, U6 USBLC6-2SC6, Y1 25MHz

Commit message: Layout V2
Parts:
- removed R2, R9: 2k2, Resistor_SMD:R_0603_1608Metric
- removed U3: 24LC512, Package_DIP:DIP-8_W7.62mm_Socket
- added U7: W25Q128JVS, Package_SO:SOIC-8_5.23x5.23mm_P1.27mm, F.Cu at (115.5, 87.5)
- C1, C2, U1: moved to F.Cu
- C15, C16, FL1, R10, U6: moved to B.Cu
- R1: value 2k2 -> 1k; moved to B.Cu
- moved C10 15.9 mm to (109.3, 90.3), turned to 180 degrees
- moved C9 13.0 mm to (109.3, 93.3), turned to 180 degrees
- moved R5 12.5 mm to (118.5, 78.1)
- moved C12 12.5 mm to (112.5, 78.1), turned to 0 degrees
- moved C7 12.5 mm to (118.9, 101.2), turned to -90 degrees
- moved SW1 11.5 mm to (117.4, 81.7), turned to -90 degrees
- moved SW2 11.5 mm to (113.6, 81.7)
- moved FL1 11.3 mm to (121.5, 114.9), turned to 0 degrees
- moved R3 10.3 mm to (115.5, 78.1)
- moved C4 10.3 mm to (114.3, 101.5), turned to 180 degrees
- moved C16 10.0 mm to (125.5, 100.9), turned to 90 degrees
- moved C1 8.81 mm to (124.8, 104.8), turned to 0 degrees
- moved R10 8.59 mm to (128.5, 100.9), turned to -90 degrees
- moved C14 8.56 mm to (106.2, 97.0), turned to 180 degrees
- moved C13 8.29 mm to (106.2, 91.2), turned to 0 degrees
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Connections:
- J2 pad 1: /SPI_NCS -> /CTRL_SPI_MOSI
- J2 pad 2: /SPI_CLK -> /CTRL_SPI_MISO
- J2 pad 3: /SPI_MISO -> /CTRL_SPI_CLK
- J2 pad 4: /SPI_MOSI -> /CTRL_SPI_NCS
- J3 pad 1: /STEPPER_A2 -> /STEPPER_B2
- J3 pad 2: /STEPPER_A1 -> /STEPPER_B1
- J3 pad 3: /STEPPER_B2 -> /STEPPER_A1
- J3 pad 4: /STEPPER_B1 -> /STEPPER_A2
- J4 pad 2: /JTAG_SWCLK -> /JTAG_SWDIO
- J4 pad 3: /JTAG_SWDIO -> /JTAG_SWCLK
- R1 pad 1: /SCL -> /TMC_UART_TX
- R1 pad 2: +3V3 -> /TMC_UART_RX
- R10 pad 2: +3.3V -> +3V3
- U4 pad 11: unconnected-(U4-PA1-Pad11) -> /TMC_MS1
- U4 pad 12: unconnected-(U4-PA2-Pad12) -> /TMC_MS2
- U4 pad 13: unconnected-(U4-PA3-Pad13) -> /TMC_NEN
- U4 pad 14: /SPI_NCS -> /CTRL_SPI_NCS
- U4 pad 15: /SPI_CLK -> /CTRL_SPI_CLK
- U4 pad 16: /SPI_MISO -> /CTRL_SPI_MISO
- U4 pad 17: /SPI_MOSI -> /CTRL_SPI_MOSI
- U4 pad 18: /TMC_STEP -> /TMC_DIAG
- U4 pad 19: /TMC_DIR -> /TMC_INDEX
- U4 pad 20: /TMC_MS1 -> unconnected-(U4-PB2-Pad20)
- U4 pad 25: unconnected-(U4-PB12-Pad25) -> /TMC_STEP
- U4 pad 26: unconnected-(U4-PB13-Pad26) -> /TMC_DIR
- U4 pad 27: unconnected-(U4-PB14-Pad27) -> /TMC_SPREAD
- U4 pad 28: unconnected-(U4-PB15-Pad28) -> /TMC_STDBY
- U4 pad 29: unconnected-(U4-PA8-Pad29) -> /STATUS
- U4 pad 30: unconnected-(U4-PA9-Pad30) -> /TMC_UART_TX
- U4 pad 31: /STATUS -> /TMC_UART_RX
- U4 pad 38: /24LC512_WP -> /FLASH_SPI_NCS
- U4 pad 39: /TMC_MS2 -> /FLASH_SPI_CLK
- U4 pad 40: /TMC_SPREAD -> /FLASH_SPI_MISO
- U4 pad 41: /TMC_STDBY -> /FLASH_SPI_MOSI
- U4 pad 42: /TMC_NDP/UART -> /W25Q128_NWP
- U4 pad 43: /TMC_DIAG -> /W25Q128_NRST
- U4 pad 45: /TMC_NEN -> unconnected-(U4-PB8-Pad45)
- U5 pad 16: unconnected-(U5-INDEX-Pad16) -> /TMC_INDEX
- U5 pad 18: /TMC_NDP/UART -> /TMC_UART_RX
Routing:
- net +24V: track 7.63 -> 49.0 mm, vias 1 -> 2
- net /TMC_NDP/UART: track 27.5 -> 0.00 mm, vias 3 -> 0
- net /SPI_MOSI: track 24.0 -> 0.00 mm, vias 1 -> 0
- net /SPI_MISO: track 22.1 -> 0.00 mm, vias 1 -> 0
- net /TMC_SPREAD: track 30.2 -> 8.89 mm
- net /TMC_INDEX: track 0.00 -> 20.9 mm, vias 0 -> 2
- net /SPI_CLK: track 20.3 -> 0.00 mm, vias 1 -> 0
- net /CTRL_SPI_NCS: track 0.00 -> 19.1 mm
- net /TMC_MS2: track 35.9 -> 17.0 mm
- net /CTRL_SPI_CLK: track 0.00 -> 18.4 mm
- net /CTRL_SPI_MISO: track 0.00 -> 17.8 mm
- net /SPI_NCS: track 17.4 -> 0.00 mm
- net /CTRL_SPI_MOSI: track 0.00 -> 17.1 mm
- net /I2C_SCL: track 18.3 -> 3.35 mm
- net /24LC512_WP: track 13.5 -> 0.00 mm, vias 1 -> 0
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- removed copper zone on In2.Cu, net +24V
- removed copper zone on B.Cu, net +3V3
Other:
- board text added: "+3v3"
- board text added: "A1"
- board text added: "A2"
- board text added: "B1"
- board text added: "B2"
- board text added: "CLK"
- board text added: "GND"
- board text added: "MISO"
- board text added: "MOSI"
- board text added: "NCS"
- board text added: "SWCLK"
- board text added: "SWDIO"
- board text removed: "-"
- board text removed: "B1 B2 A1 A2"
- board text removed: "SETTINGS"

Commit message: Silkscreen
Routing:
- net GND: vias 47 -> 87

Commit message: Updated PCB
Parts:
- FL1: value TDK ACM2012-900 -> TDK ACM2012-900; footprint ACM2012_900_2P_T002:ACM2012_TDK -> Marijn_KiCad:ACM2012_TDK_UPDATE
- J2: footprint Connector_PinHeader_2.00mm:PinHeader_1x04_P2.00mm_Vertical -> Connector_PinHeader_2.00mm:PinHeader_1x06_P2.00mm_Vertical
- U7: footprint Package_SO:SOIC-8_5.23x5.23mm_P1.27mm -> Marijn_KiCad:SOIC-8_W25QxJVS
- moved FL1 7.36 mm to (121.5, 107.5), turned to -90 degrees
- moved J2 2.00 mm to (114.5, 115.2)
Connections:
- J2 pad 1: /CTRL_SPI_MOSI -> +3V3
- J2 pad 2: /CTRL_SPI_MISO -> /CTRL_SPI_MOSI
- J2 pad 3: /CTRL_SPI_CLK -> /CTRL_SPI_MISO
- J2 pad 4: /CTRL_SPI_NCS -> /CTRL_SPI_CLK
Routing:
- net /USB_DP: track 23.5 -> 14.8 mm
- net /USB_DN: track 21.8 -> 13.6 mm
- net /USB/FL_P: track 3.22 -> 5.42 mm
- net /USB/FL_N: track 3.22 -> 5.42 mm
- net GND: vias 87 -> 89
Other:
- board text added: "STATUS"

Commit message: Update
Connections:
- U2 pad 5: GND -> unconnected-(U2-PGO-Pad5)
- U2 pad 6: /I2C_SCL -> /I2C_SDA
- U2 pad 7: /I2C_SDA -> /I2C_SCL
- U2 pad 8: unconnected-(U2-PGO-Pad8) -> GND
- U4 pad 21: /I2C_SDA -> /I2C_SCL
- U4 pad 46: /I2C_SCL -> /I2C_SDA
Routing:
- net /I2C_SDA: track 8.05 -> 3.35 mm
- net /I2C_SCL: track 3.35 -> 8.05 mm
- net GND: track 70.7 -> 71.8 mm, vias 89 -> 88
Changed lines of the file:
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@@
 	(net 18 "unconnected-(J5-SHIELD-PadS1)_2")
 	(net 19 "unconnected-(J5-SBU1-PadA8)")
-	(net 20 "unconnected-(U2-PGO-Pad8)")
+	(net 20 "unconnected-(U2-PGO-Pad5)")
 	(net 21 "unconnected-(U4-PC13-Pad2)")
 	(net 22 "/NRST")
@@
 		)
 		(fp_text user "${REFERENCE}"
-			(at 0 5 360)
+			(at 0 5 0)
 			(layer "F.Fab")
 			(effects
@@
 			(layers "F.Cu" "F.Paste" "F.Mask")
 			(roundrect_rratio 0.25)
-			(net 28 "/I2C_SDA")
+			(net 30 "/I2C_SCL")
 			(pinfunction "PB10")
 			(pintype "bidirectional")
@@
 			(net 33 "unconnected-(U4-PB8-Pad45)")
 			(pinfunction "PB8")
-			(pintype "bidirectional+no_connect")
+			(pintype "bidirectional")
 		)
 		(pad "46" smd roundrect
@@
 			(layers "F.Cu" "F.Paste" "F.Mask")
 			(roundrect_rratio 0.25)
-			(net 30 "/I2C_SCL")
+			(net 28 "/I2C_SDA")
 			(pinfunction "PB9")
 			(pintype "bidirectional")
@@
 		(fp_line
 			(start 1.95 -2.56)
-			(end 0 -2.559999)
+			(end 0 -2.56)
 			(stroke
 				(width 0.12)
@@
 		(fp_line
 			(start -1.95 -2.56)
-			(end 0 -2.559999)
+			(end 0 -2.56)
 			(stroke
 				(width 0.12)
@@
 		(fp_line
 			(start 1.95 2.56)
-			(end 0 2.559999)
+			(end 0 2.56)
 			(stroke
 				(width 0.12)
@@
 		(fp_line
 			(start -1.95 2.56)
-			(end 0 2.559999)
+			(end 0 2.56)
 			(stroke
 				(width 0.12)
@@
 		(fp_poly
 			(pts
-				(xy -2.7 2.465) (xy -2.939999 2.795) (xy -2.46 2.795) (xy -2.7 2.465)
+				(xy -2.7 2.465) (xy -2.94 2.795) (xy -2.46 2.795) (xy -2.7 2.465)
 			)
 			(stroke
@@
 		(fp_line
 			(start 1.95 2.45)
-			(end -0.975 2.450001)
+			(end -0.975 2.45)
 			(stroke
 				(width 0.1)
@@
 		)
 		(fp_line
-			(start -0.975 2.450001)
+			(start -0.975 2.45)
 			(end -1.95 1.475)
 			(stroke
@@
 			(layers "B.Cu" "B.Paste" "B.Mask")
 			(roundrect_rratio 0.25)
-			(net 1 "GND")
-			(pinfunction "DIR")
-			(pintype "input")
+			(net 20 "unconnected-(U2-PGO-Pad5)")
+			(pinfunction "PGO")
+			(pintype "input+no_connect")
 		)
 		(pad "6" smd roundrect
@@
 			(layers "B.Cu" "B.Paste" "B.Mask")
 			(roundrect_rratio 0.25)
-			(net 30 "/I2C_SCL")
-			(pinfunction "SCL")
-			(pintype "input")
+			(net 28 "/I2C_SDA")
+			(pinfunction "SDA")
+			(pintype "bidirectional")
 		)
 		(pad "7" smd roundrect
@@
 			(layers "B.Cu" "B.Paste" "B.Mask")
 			(roundrect_rratio 0.25)
-			(net 28 "/I2C_SDA")
-			(pinfunction "SDA")
-			(pintype "bidirectional")
+			(net 30 "/I2C_SCL")
+			(pinfunction "SCL")
+			(pintype "input")
 		)
 		(pad "8" smd roundrect
@@
 			(layers "B.Cu" "B.Paste" "B.Mask")
 			(roundrect_rratio 0.25)
-			(net 20 "unconnected-(U2-PGO-Pad8)")
-			(pinfunction "PGO")
-			(pintype "input+no_connect")
+			(net 1 "GND")
+			(pinfunction "DIR")
+			(pintype "input")
 		)
 		(model "${KICAD8_3DMODEL_DIR}/Package_SO.3dshapes/SOIC-8_3.9x4.9mm_P1.27mm.wrl"
@@
 	)
 	(via
-		(at 113.1 93.1)
-		(size 0.6)
-		(drill 0.3)
-		(layers "F.Cu" "B.Cu")
-		(net 1)
-	)
-	(via
 		(at 135.5 105.5)
 		(size 0.6)
@@
 	)
 	(segment
-		(start 113.175 93.025)
-		(end 113.1 93.1)
+		(start 117.405 94.005)
+		(end 117.9 94.5)
 		(width 0.5)
 		(layer "B.Cu")
@@
 	)
 	(segment
+		(start 117.405 93.025)
+		(end 117.405 94.005)
+		(width 0.5)
+		(layer "B.Cu")
+		(net 1)
+	)
+	(segment
 		(start 113.595 97.975)
 		(end 113.595 99.955)
@@
 	)
 	(segment
-		(start 113.595 93.025)
-		(end 113.175 93.025)
-		(width 0.5)
-		(layer "B.Cu")
-		(net 1)
-	)
-	(segment
 		(start 119.1 108.705)
 		(end 119.3 108.905)
@@
 	)
 	(segment
-		(start 116.75 99.554433)
-		(end 116.75 98.9375)
+		(start 113.75 91.15)
+		(end 113.8 91.1)
 		(width 0.2)
 		(layer "F.Cu")
@@
 	)
 	(segment
-		(start 116.507512 99.796921)
-		(end 116.75 99.554433)
+		(start 113.75 92.0625)
+		(end 113.75 91.15)
 		(width 0.2)
 		(layer "F.Cu")
@@
 	)
 	(via
-		(at 116.507512 99.796921)
+		(at 113.8 91.1)
 		(size 0.6)
 		(drill 0.3)
@@
 	)
 	(segment
-		(start 116.507512 99.796921)
-		(end 116.7 99.604433)
-		(width 0.2)
-		(layer "B.Cu")
-		(net 28)
-	)
-	(segment
-		(start 116.7 93.59)
-		(end 116.135 93.025)
+		(start 114.865 92.165)
+		(end 113.8 91.1)
 		(width 0.2)
 		(layer "B.Cu")
@@
 	)
 	(segment
-		(start 116.7 99.604433)
-		(end 116.7 93.59)
+		(start 114.865 93.025)
+		(end 114.865 92.165)
 		(width 0.2)
 		(layer "B.Cu")
@@
 	)
 	(segment
-		(start 113.75 91.15)
-		(end 113.8 91.1)
+		(start 116.75 99.554433)
+		(end 116.75 98.9375)
 		(width 0.2)
 		(layer "F.Cu")
@@
 	)
 	(segment
-		(start 113.75 92.0625)
-		(end 113.75 91.15)
+		(start 116.507512 99.796921)
+		(end 116.75 99.554433)
 		(width 0.2)
 		(layer "F.Cu")
@@
 	)
 	(via
-		(at 113.8 91.1)
+		(at 116.507512 99.796921)
 		(size 0.6)
 		(drill 0.3)
@@
 	)
 	(segment
-		(start 114.865 92.165)
-		(end 113.8 91.1)
+		(start 116.507512 99.796921)
+		(end 116.7 99.604433)
 		(width 0.2)
 		(layer "B.Cu")
@@
 	)
 	(segment
-		(start 114.865 93.025)
-		(end 114.865 92.165)
+		(start 116.7 93.59)
+		(end 116.135 93.025)
+		(width 0.2)
+		(layer "B.Cu")
+		(net 30)
+	)
+	(segment
+		(start 116.7 99.604433)
+		(end 116.7 93.59)
 		(width 0.2)
 		(layer "B.Cu")
@@
 		(hatch edge 0.5)
 		(connect_pads yes
-			(clearance 0.5)
+			(clearance 0.2)
 		)
-		(min_thickness 0.25)
+		(min_thickness 0.2)
 		(filled_areas_thickness no)
 		(fill yes
@@
 		(priority 1)
 		(connect_pads
-			(clearance 0.5)
+			(clearance 0.2)
 		)
-		(min_thickness 0.25)
+		(min_thickness 0.2)
 		(filled_areas_thickness no)
 		(fill yes
@@
 		(hatch edge 0.5)
 		(connect_pads yes
-			(clearance 0.5)
+			(clearance 0.2)
 		)
-		(min_thickness 0.25)
+		(min_thickness 0.2)
 		(filled_areas_thickness no)
 		(fill yes
@@
 		(hatch edge 0.5)
 		(connect_pads yes
-			(clearance 0.5)
+			(clearance 0.2)
 		)
-		(min_thickness 0.25)
+		(min_thickness 0.2)
 		(filled_areas_thickness no)
 		(fill yes
@@
 		(hatch edge 0.5)
 		(connect_pads yes
-			(clearance 0.5)
+			(clearance 0.2)
 		)
-		(min_thickness 0.25)
+		(min_thickness 0.2)
 		(filled_areas_thickness no)
 		(fill yes
