File: stepper_driver_PCB/stepper_driver_PCB.kicad_sch (KiCad schematic)
At the start: 42 parts, among them J1 POWER, J2 CTRL, J3 STEPPER, J4 JTAG, SW1 BTN, SW2 BTN, U1 AP7343, U4 STM32F412CEUx, U5 TMC2226-SA, U7 W25Q128JVS, Y1 25MHz

Commit message: Updated PCB
Parts:
- removed J2: CTRL, Connector_PinHeader_2.00mm:PinHeader_1x04_P2.00mm_Vertical, symbol Connector_Generic:Conn_01x04
- added J2: CTRL, Connector_PinHeader_2.00mm:PinHeader_1x06_P2.00mm_Vertical, symbol Connector_Generic:Conn_01x06
- U7: footprint Package_SO:SOIC-8_5.23x5.23mm_P1.27mm -> Marijn_KiCad:SOIC-8_W25QxJVS
Connections:
- net +3V3: now also J2.1 (Pin_1)
- net CTRL_SPI_CLK: now also J2.4 (Pin_4)
- net CTRL_SPI_MISO: now also J2.3 (Pin_3)
- net CTRL_SPI_MOSI: now also J2.2 (Pin_2)
- net CTRL_SPI_NCS: now also J2.5 (Pin_5)
- net GND: now also J2.6 (Pin_6)
- no-connect marks 6 -> 7
Changed lines of the file:
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@@
 		(at 210.82 63.5)
 	)
+	(no_connect
+		(at 40.64 86.36)
+	)
 	(wire
 		(pts
@@
 	(wire
 		(pts
-			(xy 172.72 25.4) (xy 172.72 24.13)
+			(xy 172.72 26.67) (xy 172.72 25.4)
 		)
 		(stroke
@@
 	(wire
 		(pts
+			(xy 171.45 19.05) (xy 171.45 20.32)
+		)
+		(stroke
+			(width 0)
+			(type default)
+		)
+	)
+	(wire
+		(pts
 			(xy 57.15 130.81) (xy 58.42 130.81)
 		)
@@
 	(wire
 		(pts
-			(xy 172.72 22.86) (xy 172.72 21.59)
+			(xy 172.72 24.13) (xy 172.72 22.86)
 		)
 		(stroke
@@
 	(wire
 		(pts
+			(xy 171.45 33.02) (xy 172.72 33.02)
+		)
+		(stroke
+			(width 0)
+			(type default)
+		)
+	)
+	(wire
+		(pts
 			(xy 113.03 85.09) (xy 121.92 85.09)
 		)
@@
 	(wire
 		(pts
-			(xy 172.72 30.48) (xy 172.72 29.21)
+			(xy 172.72 31.75) (xy 172.72 30.48)
 		)
 		(stroke
@@
 	(wire
 		(pts
+			(xy 171.45 34.29) (xy 171.45 33.02)
+		)
+		(stroke
+			(width 0)
+			(type default)
+		)
+	)
+	(wire
+		(pts
 			(xy 121.92 97.79) (xy 121.92 96.52)
 		)
@@
 	(wire
 		(pts
-			(xy 172.72 27.94) (xy 172.72 26.67)
+			(xy 172.72 29.21) (xy 172.72 27.94)
 		)
 		(stroke
@@
 	(wire
 		(pts
+			(xy 171.45 20.32) (xy 172.72 20.32)
+		)
+		(stroke
+			(width 0)
+			(type default)
+		)
+	)
+	(wire
+		(pts
 			(xy 53.34 46.99) (xy 55.88 46.99)
 		)
@@
 	)
 	(label "CTRL_SPI_MOSI"
-		(at 172.72 22.86 180)
+		(at 172.72 24.13 180)
 		(fields_autoplaced yes)
 		(effects
@@
 	)
 	(label "CTRL_SPI_MISO"
-		(at 172.72 25.4 180)
+		(at 172.72 26.67 180)
 		(fields_autoplaced yes)
 		(effects
@@
 	)
 	(label "CTRL_SPI_CLK"
-		(at 172.72 27.94 180)
+		(at 172.72 29.21 180)
 		(fields_autoplaced yes)
 		(effects
@@
 	)
 	(label "CTRL_SPI_NCS"
-		(at 172.72 30.48 180)
+		(at 172.72 31.75 180)
 		(fields_autoplaced yes)
 		(effects
@@
 			)
 		)
-		(property "Footprint" "Package_SO:SOIC-8_5.23x5.23mm_P1.27mm"
+		(property "Footprint" "Marijn_KiCad:SOIC-8_W25QxJVS"
 			(at 212.09 115.57 0)
 			(effects
@@
 		)
 		(property "Value" "10u"
-			(at 83.82 177.8 90)
+			(at 85.344 178.054 90)
 			(effects
 				(font
@@
 	)
 	(symbol
+		(lib_id "Connector_Generic:Conn_01x06")
+		(at 177.8 25.4 0)
+		(unit 1)
+		(exclude_from_sim no)
+		(in_bom yes)
+		(on_board yes)
+		(dnp no)
+		(property "Reference" "J2"
+			(at 176.53 17.78 0)
+			(effects
+				(font
+					(size 1.27 1.27)
+				)
+				(justify left)
+			)
+		)
+		(property "Value" "CTRL"
+			(at 175.514 35.56 0)
+			(effects
+				(font
+					(size 1.27 1.27)
+				)
+				(justify left)
+			)
+		)
+		(property "Footprint" "Connector_PinHeader_2.00mm:PinHeader_1x06_P2.00mm_Vertical"
+			(at 177.8 25.4 0)
+			(effects
+				(font
+					(size 1.27 1.27)
+				)
+				(hide yes)
+			)
+		)
+		(property "Datasheet" "~"
+			(at 177.8 25.4 0)
+			(effects
+				(font
+					(size 1.27 1.27)
+				)
+				(hide yes)
+			)
+		)
+		(property "Description" "Generic connector, single row, 01x06, script generated (kicad-library-utils/schlib/autogen/connector/)"
+			(at 177.8 25.4 0)
+			(effects
+				(font
+					(size 1.27 1.27)
+				)
+				(hide yes)
+			)
+		)
+		(pin "4"
+		)
+		(pin "3"
+		)
+		(pin "2"
+		)
+		(pin "1"
+		)
+		(pin "6"
+		)
+		(pin "5"
+		)
+		(instances
+			(project ""
+				(path "/55e5f9ee-4ad9-4c00-8411-66894e392a47"
+					(reference "J2")
+					(unit 1)
+				)
+			)
+		)
+	)
+	(symbol
 		(lib_id "Switch:SW_Push")
 		(at 144.78 180.34 270)
@@
 	)
 	(symbol
-		(lib_id "Connector_Generic:Conn_01x04")
-		(at 177.8 24.13 0)
-		(unit 1)
-		(exclude_from_sim no)
-		(in_bom yes)
-		(on_board yes)
-		(dnp no)
-		(property "Reference" "J2"
-			(at 176.53 19.05 0)
-			(effects
-				(font
-					(size 1.27 1.27)
-				)
-				(justify left)
-			)
-		)
-		(property "Value" "CTRL"
-			(at 175.514 32.004 0)
-			(effects
-				(font
-					(size 1.27 1.27)
-				)
-				(justify left)
-			)
-		)
-		(property "Footprint" "Connector_PinHeader_2.00mm:PinHeader_1x04_P2.00mm_Vertical"
-			(at 177.8 24.13 0)
-			(effects
-				(font
-					(size 1.27 1.27)
-				)
-				(hide yes)
-			)
-		)
-		(property "Datasheet" "~"
-			(at 177.8 24.13 0)
-			(effects
-				(font
-					(size 1.27 1.27)
-				)
-				(hide yes)
-			)
-		)
-		(property "Description" "Generic connector, single row, 01x04, script generated (kicad-library-utils/schlib/autogen/connector/)"
-			(at 177.8 24.13 0)
-			(effects
-				(font
-					(size 1.27 1.27)
-				)
-				(hide yes)
-			)
-		)
-		(pin "2"
-		)
-		(pin "1"
-		)
-		(pin "3"
-		)
-		(pin "4"
-		)
-		(instances
-			(project ""
-				(path "/55e5f9ee-4ad9-4c00-8411-66894e392a47"
-					(reference "J2")
-					(unit 1)
-				)
-			)
-		)
-	)
-	(symbol
 		(lib_id "power:GND")
 		(at 121.92 78.74 270)
@@
 	)
 	(symbol
+		(lib_id "power:+3V3")
+		(at 171.45 19.05 0)
+		(unit 1)
+		(exclude_from_sim no)
+		(in_bom yes)
+		(on_board yes)
+		(dnp no)
+		(property "Reference" "#PWR024"
+			(at 171.45 22.86 0)
+			(effects
+				(font
+					(size 1.27 1.27)
+				)
+				(hide yes)
+			)
+		)
+		(property "Value" "+3V3"
+			(at 171.45 15.24 0)
+			(effects
+				(font
+					(size 1.27 1.27)
+				)
+			)
+		)
+		(property "Footprint" ""
+			(at 171.45 19.05 0)
+			(effects
+				(font
+					(size 1.27 1.27)
+				)
+				(hide yes)
+			)
+		)
+		(property "Datasheet" ""
+			(at 171.45 19.05 0)
+			(effects
+				(font
+					(size 1.27 1.27)
+				)
+				(hide yes)
+			)
+		)
+		(property "Description" "Power symbol creates a global label with name \"+3V3\""
+			(at 171.45 19.05 0)
+			(effects
+				(font
+					(size 1.27 1.27)
+				)
+				(hide yes)
+			)
+		)
+		(pin "1"
+		)
+		(instances
+			(project "stepper_driver_PCB"
+				(path "/55e5f9ee-4ad9-4c00-8411-66894e392a47"
+					(reference "#PWR024")
+					(unit 1)
+				)
+			)
+		)
+	)
+	(symbol
 		(lib_id "power:GND")
 		(at 111.76 184.15 0)
@@
 					(unit 1)
 				)
+			)
+		)
+	)
+	(symbol
+		(lib_id "power:GND")
+		(at 171.45 34.29 0)
+		(unit 1)
+		(exclude_from_sim no)
+		(in_bom yes)
+		(on_board yes)
+		(dnp no)
+		(property "Reference" "#PWR023"
+			(at 171.45 40.64 0)
+			(effects
+				(font
+					(size 1.27 1.27)
+				)
+				(hide yes)
+			)
+		)
+		(property "Value" "GND"
+			(at 170.434 38.354 0)
+			(effects
+				(font
+					(size 1.27 1.27)
+				)
+			)
+		)
+		(property "Footprint" ""
+			(at 171.45 34.29 0)
+			(effects
+				(font
+					(size 1.27 1.27)
+				)
+				(hide yes)
+			)
+		)
+		(property "Datasheet" ""
+			(at 171.45 34.29 0)
+			(effects
+				(font
+					(size 1.27 1.27)
+				)
+				(hide yes)
+			)
+		)
+		(property "Description" "Power symbol creates a global label with name \"GND\" , ground"
+			(at 171.45 34.29 0)
+			(effects
+				(font
+					(size 1.27 1.27)
+				)
+				(hide yes)
+			)
+		)
+		(pin "1"
+		)
+		(instances
+			(project "stepper_driver_PCB"
+				(path "/55e5f9ee-4ad9-4c00-8411-66894e392a47"
+					(reference "#PWR023")
+					(unit 1)
+				)

Commit message: Update
Connections:
- net GND: now also U2.8 (DIR); no longer U2.5 (DIR)
- net I2C_SCL: now also U2.7 (SCL), U4.21 (PB10); no longer U2.6 (SCL), U4.46 (PB9)
- net I2C_SDA: now also U2.6 (SDA), U4.46 (PB9); no longer U2.7 (SDA), U4.21 (PB10)
- no-connect marks 7 -> 6
Changed lines of the file:
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@@
-	)
-	(no_connect
-		(at 40.64 101.6)
 	)
 	(no_connect
@@
 	(wire
 		(pts
+			(xy 40.64 105.41) (xy 40.64 104.14)
+		)
+		(stroke
+			(width 0)
+			(type default)
+		)
+	)
+	(wire
+		(pts
 			(xy 152.4 85.09) (xy 152.4 83.82)
 		)
@@
 	(wire
 		(pts
-			(xy 40.64 105.41) (xy 40.64 104.14)
-		)
-		(stroke
-			(width 0)
-			(type default)
-		)
-	)
-	(wire
-		(pts
 			(xy 201.93 116.84) (xy 201.93 115.57)
 		)
@@
 	(wire
 		(pts
+			(xy 40.64 107.95) (xy 40.64 106.68)
+		)
+		(stroke
+			(width 0)
+			(type default)
+		)
+	)
+	(wire
+		(pts
 			(xy 58.42 46.99) (xy 58.42 48.26)
 		)
@@
 		(pts
 			(xy 31.75 185.42) (xy 31.75 187.96)
-		)
-		(stroke
-			(width 0)
-			(type default)
-		)
-	)
-	(wire
-		(pts
-			(xy 40.64 107.95) (xy 40.64 106.68)
 		)
 		(stroke
@@
 	(text "I2C"
 		(exclude_from_sim no)
-		(at 20.574 105.664 90)
+		(at 22.86 105.41 90)
 		(effects
 			(font
@@
 	)
 	(label "I2C_SCL"
-		(at 40.64 105.41 180)
+		(at 40.64 107.95 180)
 		(fields_autoplaced yes)
 		(effects
@@
 	)
 	(label "I2C_SDA"
-		(at 40.64 107.95 180)
-		(fields_autoplaced yes)
-		(effects
+		(at 40.64 105.41 180)
+		(fields_autoplaced yes)
+		(effects
